Commit message: Add back in joint limits, broken without

File: urdf/helix.xacro (robot description, xacro)
@@ -2,5 +2,5 @@
 <robot xmlns:xacro="http://ros.org/wiki/xacro">
 <!-- Very basic representation of Helix motor base and pulleys -->
-<!-- TODO - effort/velocity limits taken from dynamixel_hardware_examples package, not sure what they correpsond to wrt current-->
+<!-- TODO - effort/velocity limits taken from dynamixel_hardware_examples package, not sure what they correpsond to wrt current -->
 <material name='black'>
   <color rgba="0.2 0.2 0.2 1.0"/>
@@ -46,5 +46,5 @@
     <origin xyz="-0.043 0.025 0.12" rpy="0 0 4.2"/>
     <axis xyz="1 0 0"/>
-    <limit velocity="4.8" effort="1"/>
+    <limit velocity="4.8" effort="1" lower="-3.0" upper="3.0" />
   </joint>
    <!-- Link 0 -->
@@ -64,5 +64,5 @@
     <origin xyz="0 -0.05 0.12" rpy="0 0 0"/>
     <axis xyz="1 0 0"/>
-    <limit velocity="4.8" effort="1"/>
+    <limit velocity="4.8" effort="1" lower="-3.0" upper="3.0" />
   </joint>
    <!-- Link 1 -->
@@ -82,5 +82,5 @@
     <origin xyz="0.043 0.025 0.12" rpy="0 0 2.1"/>
     <axis xyz="1 0 0"/>
-    <limit velocity="4.8" effort="1"/>
+    <limit velocity="4.8" effort="1" lower="-3.0" upper="3.0" />
   </joint>
    <!-- Link 2 -->
@@ -100,5 +100,5 @@
     <origin xyz="0.16 0 0.025" rpy="0 0 0"/>
     <axis xyz="1 0 0"/>
-    <limit velocity="4.8" effort="1"/>
+    <limit velocity="4.8" effort="1" lower="-3.0" upper="3.0" />
   </joint>
    <!-- Link 3 -->
@@ -118,5 +118,5 @@
     <origin xyz="-0.08 0.138 0.025" rpy="0 0 2.1"/>
     <axis xyz="1 0 0"/>
-    <limit velocity="4.8" effort="1"/>
+    <limit velocity="4.8" effort="1" lower="-3.0" upper="3.0" />
   </joint>
    <!-- Link 4 -->
@@ -136,5 +136,5 @@
     <origin xyz="-0.08 -0.138 0.025" rpy="0 0 4.2"/>
     <axis xyz="1 0 0"/>
-    <limit velocity="4.8" effort="1"/>
+    <limit velocity="4.8" effort="1" lower="-3.0" upper="3.0" />
   </joint>
    <!-- Link 5 -->
@@ -154,5 +154,5 @@
     <origin xyz="0.08 -0.138 0.025" rpy="0 0 5.2"/>
     <axis xyz="1 0 0"/>
-    <limit velocity="4.8" effort="1"/>
+    <limit velocity="4.8" effort="1" lower="-3.0" upper="3.0" />
   </joint>
    <!-- Link 6 -->
@@ -172,5 +172,5 @@
     <origin xyz="0.08 0.138 0.025" rpy="0 0 1.0"/>
     <axis xyz="1 0 0"/>
-    <limit velocity="4.8" effort="1"/>
+    <limit velocity="4.8" effort="1" lower="-3.0" upper="3.0" />
   </joint>
    <!-- Link 7 -->
@@ -190,5 +190,5 @@
     <origin xyz="-0.16 0 0.025" rpy="0 0 3.1"/>
     <axis xyz="1 0 0"/>
-    <limit velocity="4.8" effort="1"/>
+    <limit velocity="4.8" effort="1" lower="-3.0" upper="3.0" />
   </joint>
    <!-- Link 8 -->
